File: schematic/gpsdo/gpsdo.kicad_pcb (KiCad board)
At the start: 2 copper layers, 22.9 x 20.3 mm, 16 parts, among them J1 Conn_01x01_Male, J2 Conn_01x01_Male, J3 Conn_01x01_Male, J4 Conn_01x01_Male, U1 74HC04, Y1 10MHz

Commit message: Add text on board to satisfy pcb fab
Other:
- board text added: "GPSDO"
Changed lines of the file:
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@@
-(kicad_pcb (version 20171130) (host pcbnew 5.0.0)
+(kicad_pcb (version 20171130) (host pcbnew 5.1.5)
   (general
     (thickness 1.6)
-    (drawings 4)
+    (drawings 5)
     (tracks 52)
     (zones 0)
@@
     (zone_45_only no)
     (trace_min 0.3)
-    (segment_width 0.2)
-    (edge_width 0.15)
     (via_size 0.8)
     (via_drill 0.4)
@@
     (uvia_min_size 0.2)
     (uvia_min_drill 0.1)
+    (edge_width 0.15)
+    (segment_width 0.2)
     (pcb_text_width 0.3)
     (pcb_text_size 1.5 1.5)
@@
     (uvia_dia 0.3)
     (uvia_drill 0.1)
+    (diff_pair_width 0.3)
     (diff_pair_gap 0.25)
-    (diff_pair_width 0.3)
     (add_net +5V)
     (add_net GND)
@@
     )
   )
+  (gr_text GPSDO (at 48.26 177.546) (layer B.Cu)
+    (effects (font (size 0.5 0.5) (thickness 0.125)) (justify mirror))
+  )
   (gr_line (start 57.15 161.29) (end 34.29 161.29) (layer Edge.Cuts) (width 0.15))

Commit message: Update GPSDO schematic to used values
Parts:
- C4: value 68p -> 10p
- R2: value 470k -> 1M
Changed lines of the file:
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@@
       (effects (font (size 1 1) (thickness 0.15)) (justify mirror))
     )
-    (fp_text value 68p (at 0 -1.65 270) (layer B.Fab)
+    (fp_text value 10p (at 0 -1.65 270) (layer B.Fab)
       (effects (font (size 1 1) (thickness 0.15)) (justify mirror))
     )
@@
       (effects (font (size 1 1) (thickness 0.15)) (justify mirror))
     )
-    (fp_text value 470k (at 0 -1.65 270) (layer B.Fab)
-      (effects (font (size 1 1) (thickness 0.15)) (justify mirror))
-    )
+    (fp_text value 1M (at 0 -1.65 270) (layer B.Fab)
+      (effects (font (size 1 1) (thickness 0.15)) (justify mirror))
+    )
