File: schematic/gpsdo/gpsdo.sch (KiCad schematic (older format))
At the start: 16 parts, among them J1 Conn_01x01_Male, J2 Conn_01x01_Male, J3 Conn_01x01_Male, J4 Conn_01x01_Male, U1 74HC04, Y1 10MHz

Commit message: Update GPSDO schematic to used values
Parts:
- C4: value 68p -> 10p
- R2: value 470k -> 1M
Changed lines of the file:
@@
 EESchema Schematic File Version 4
-LIBS:gpsdo-cache
-EELAYER 26 0
+EELAYER 30 0
 EELAYER END
 $Descr A4 11693 8268
@@
 P 2100 3850
 F 0 "C4" H 2215 3896 50  0000 L CNN
-F 1 "68p" H 2215 3805 50  0000 L CNN
+F 1 "10p" H 2215 3805 50  0000 L CNN
 F 2 "Capacitor_SMD:C_0805_2012Metric_Pad1.15x1.40mm_HandSolder" H 2138 3700 50  0001 C CNN
 F 3 "~" H 2100 3850 50  0001 C CNN
@@
 P 2800 3800
 F 0 "R2" V 2593 3800 50  0000 C CNN
-F 1 "470k" V 2684 3800 50  0000 C CNN
+F 1 "1M" V 2684 3800 50  0000 C CNN
 F 2 "Resistor_SMD:R_0805_2012Metric_Pad1.15x1.40mm_HandSolder" V 2730 3800 50  0001 C CNN
 F 3 "~" H 2800 3800 50  0001 C CNN
