File: schematic/tray1/tray1.kicad_pcb (KiCad board)
At the start: 2 copper layers, 49.5 x 100.3 mm, 15 parts, among them J1 Conn_02x10_Odd_Even, J2 Conn_02x05_Odd_Even, J3 Conn_Coaxial, U1 ATmega128-16AU, U2 GPS, U3 ST485EBDR, U4 74HC04, Y1 TXCO

Commit message: Add separate regulator for low noise
Parts:
- added C6: 100n, Capacitor_SMD:C_0805_2012Metric_Pad1.15x1.40mm_HandSolder, B.Cu at (34.1, 161.6)
- added U5: LM1117-5.0, Package_TO_SOT_SMD:SOT-223-3_TabPin2, B.Cu at (42.5, 164.4)
Connections:
- J1 pad 3: VCC -> Net-(J1-Pad3)
Routing:
- net VCC: track 164.3 -> 179.9 mm
- net Net-(C6-Pad1): track 0.00 -> 9.44 mm
